File: PCB-first/PCB-first.kicad_pcb (KiCad board)
At the start: 2 copper layers, 40.5 x 64.3 mm, 7 parts, among them SW1 SW_Push, SW2 SW_Push, SW3 SW_Push, SW4 SW_Push, U1 XIAO-RP2040-DIP

Commit message: fixed 5v net
Connections:
- net Net-(D1-VDD) renamed +5V
